File: joysticktester.sch (KiCad schematic (older format))
At the start: 18 parts, among them J1 USB_OTG, J2 DB9_Male

Commit message: fix led connection
Connections:
- net GROUND: no longer R1.2, R2.2, R3.2, R4.2, R5.2, R6.2, R7.2
- net VCC: now also R1.2, R2.2, R3.2, R4.2, R5.2, R6.2, R7.2
Changed lines of the file:
@@
 Comp "Alessio Garzi"
 Comment1 "Simple db9 joystick tester for Amiga and C64GS computers"
-Comment2 ""
-Comment3 ""
+Comment2 "Leds - 2v 20mA"
+Comment3 "Resistors 150 OHM"
 Comment4 ""
 $EndDescr
@@
 	5700 4700 5850 4700
 Text Label 5200 4400 2    60   ~ 0
-GROUND
+VCC
 Text Label 5200 4700 2    60   ~ 0
-GROUND
+VCC
 Text Label 5200 4100 2    60   ~ 0
-GROUND
+VCC
 Wire Wire Line
 	5400 3800 5200 3800
 Text Label 5200 3800 2    60   ~ 0
-GROUND
+VCC
 $Comp
 L R R5
@@
 	6150 5300 6450 5300
 Text Label 5200 5000 2    60   ~ 0
-GROUND
+VCC
 Text Label 5200 5300 2    60   ~ 0
-GROUND
+VCC
 Wire Wire Line
 	5000 2100 5000 2200
@@
 NoConn ~ 1550 2150
 $Comp
-L PWR_FLAG #FLG01
+L PWR_FLAG #FLG2
 U 1 1 5A8E78FF
 P 1950 1000
-F 0 "#FLG01" H 1950 1075 50  0001 C CNN
+F 0 "#FLG2" H 1950 1075 50  0001 C CNN
 F 1 "PWR_FLAG" H 1950 1150 50  0000 C CNN
 F 2 "" H 1950 1000 50  0001 C CNN
@@
 VCC
 $Comp
-L PWR_FLAG #FLG02
+L PWR_FLAG #FLG1
 U 1 1 5A8E7AD1
 P 1350 1000
-F 0 "#FLG02" H 1350 1075 50  0001 C CNN
+F 0 "#FLG1" H 1350 1075 50  0001 C CNN
 F 1 "PWR_FLAG" H 1350 1150 50  0000 C CNN
 F 2 "" H 1350 1000 50  0001 C CNN
@@
 	6150 5600 6450 5600
 Text Label 5200 5600 2    60   ~ 0
-GROUND
+VCC
 Text Label 6450 5600 0    60   ~ 0
 BUTTON3

Commit message: new db9 connector
Parts:
- removed J2: DB9_Male, Connectors_DSub:DSUB-9_Male_Horizontal_Pitch2.77x2.54mm_EdgePinOffset9.40mm, symbol DB9_Male
- added J3: DB-9, w_conn_d-sub:DB_9M, symbol DB-9
Connections:
- net BUTTON1: now also J3.9
- net BUTTON2: now also J3.6
- net BUTTON3: now also J3.5
- net DOWN: now also J3.2
- net GROUND: now also J3.8
- net LEFT: now also J3.3
- net RIGHT: now also J3.4
- net UP: now also J3.1
- net VCC: now also J3.7
Other:
- moved on the sheet: D1, D2, D3, D4, D5, D6, D7, D8, R1, R2, R3, R4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
